Commit message: Tuning params for HeROS map, removing wheels visualization

File: minirys_description/src/description/minirys_description.urdf (robot description, URDF)
Before this commit: robot minirys, 8 links, 13 joints
Joints:
- joint base_link_to_leftwheel_joint: type continuous -> fixed
- joint base_link_to_rightwheel_joint: type continuous -> fixed
- joint robot_base_joint: type fixed -> continuous

Commit message: Multirobot navigation

File: minirys_description/src/description/minirys_description.urdf (robot description, URDF)
Before this commit: robot minirys, 8 links, 13 joints
Links:
- removed link base_footprint
- removed link base_link
- removed link imu
- removed link laser_scan
- removed link leftwheel
- removed link rightwheel
- removed link robot_base
- removed link robot_frame
- added link $(arg namespace)/base_footprint
- added link $(arg namespace)/base_link
- added link $(arg namespace)/imu, mass 0.005; collision box size=0.003 0.010 0.023; visual box size=0.003 0.010 0.023
- added link $(arg namespace)/laser_scan, mass 0.005; collision box size=0.002 0.018 0.013; visual mesh filename=package://minirys_description/src/description/stl/LD06_lida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
- added link $(arg namespace)/leftwheel, mass ${wheel_mass}; collision cylinder length=0.015 radius=0.055463; visual mesh filename=package://minirys_description/src/description/stl/wheelpop.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
- added link $(arg namespace)/rightwheel, mass ${wheel_mass}; collision cylinder length=0.015 radius=0.055463; visual mesh filename=package://minirys_description/src/description/stl/wheelpop.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
- added link $(arg namespace)/robot_base, mass ${body_mass}; collision box size=0.07 0.116 0.13; collision cylinder length=0.01 radius=0.067
- added link $(arg namespace)/robot_frame; visual mesh filename=package://minirys_description/src/description/stl/frame_coo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
Joints:
- removed joint base_frame_joint
- removed joint base_joint
- removed joint base_link_to_leftwheel_joint
- removed joint base_link_to_rightwheel_joint
- removed joint distance_0_joint
- removed joint distance_1_joint
- removed joint distance_2_joint
- removed joint distance_3_joint
- removed joint distance_4_joint
- removed joint distance_5_joint
- removed joint imu_joint
- removed joint laser_scan_joint
- removed joint robot_base_joint
- added joint $(arg namespace)/base_footprint_joint: type fixed, parent $(arg namespace)/base_footprint, child $(arg namespace)/base_link, origin xyz=0.0 0.0 ${wheel_radius} rpy=0 0 0
- added joint $(arg namespace)/base_frame_joint: type fixed, parent $(arg namespace)/robot_base, child $(arg namespace)/robot_frame, origin xyz=0 0 0 rpy=0 0 0
- added joint $(arg namespace)/base_link_to_leftwheel_joint: type fixed, parent $(arg namespace)/base_link, child $(arg namespace)/leftwheel, origin xyz=0 -${wheel_yoff} 0 rpy=0 0 0, axis 0 -1 0
- added joint $(arg namespace)/base_link_to_rightwheel_joint: type fixed, parent $(arg namespace)/base_link, child $(arg namespace)/rightwheel, origin xyz=0 ${wheel_yoff} 0 rpy=0 0 3.14159, axis 0 -1 0
- added joint $(arg namespace)/distance_0_joint: type fixed, parent $(arg namespace)/robot_base, child $(arg namespace)/distance_0, origin xyz=0.093 -0.040 0 rpy=0 0 0
- added joint $(arg namespace)/distance_1_joint: type fixed, parent $(arg namespace)/robot_base, child $(arg namespace)/distance_1, origin xyz=-0.022 0 -0.021 rpy=3.14159 0 3.14159
- added joint $(arg namespace)/distance_2_joint: type fixed, parent $(arg namespace)/robot_base, child $(arg namespace)/distance_2, origin xyz=0.06 0.050 0 rpy=1.5708 0 1.5708
- added joint $(arg namespace)/distance_3_joint: type fixed, parent $(arg namespace)/robot_base, child $(arg namespace)/distance_3, origin xyz=0.061 0 0.030 rpy=3.14159 -1.5708 0
- added joint $(arg namespace)/distance_4_joint: type fixed, parent $(arg namespace)/robot_base, child $(arg namespace)/distance_4, origin xyz=0.061 0 -0.030 rpy=0 1.5708 0
- added joint $(arg namespace)/distance_5_joint: type fixed, parent $(arg namespace)/robot_base, child $(arg namespace)/distance_5, origin xyz=0.06 -0.050 0 rpy=-1.5708 0 -1.5708
- added joint $(arg namespace)/imu_joint: type fixed, parent $(arg namespace)/robot_base, child $(arg namespace)/imu, origin xyz=0 0 0 rpy=0 0 0
- added joint $(arg namespace)/laser_scan_joint: type fixed, parent $(arg namespace)/robot_base, child $(arg namespace)/laser_scan, origin xyz=0.044 0 0.059 rpy=0 0 0
- added joint $(arg namespace)/robot_base_joint: type continuous, parent $(arg namespace)/base_link, child $(arg namespace)/robot_base, origin xyz=0 0 0 rpy=0 0 0

Commit message: Swarm behaviour fixes

File: minirys_description/src/description/minirys_description.urdf (robot description, URDF)
Before this commit: robot minirys, 8 links, 13 joints
Joints:
- removed joint $(arg namespace)/distance_0_joint
- removed joint $(arg namespace)/distance_1_joint
- removed joint $(arg namespace)/distance_2_joint
- removed joint $(arg namespace)/distance_3_joint
- removed joint $(arg namespace)/distance_4_joint
- removed joint $(arg namespace)/distance_5_joint
